Commit message: Changes

File: wsg_50_simulation/urdf/wsg50.urdf.xacro (robot description, xacro)
@@ -1,10 +1,8 @@
 <?xml version="1.0"?>
 <robot name="wsg50" xmlns:xacro="http://www.ros.org/wiki/xacro">
-    <xacro:arg name="real_hardware" default="false"/>
-    <xacro:arg name="sim_standalone" default="true"/>
     <!-- Import wsg50 macro -->
     <xacro:include filename="$(find wsg_50_simulation)/urdf/wsg_50.urdf.xacro" />
     <link name="base_link"/>
-    <xacro:wsg_50_xacro prefix="wsg50" parent="base_link" finger_length="0.023" finger_tip="0.0" sim_standalone="$(arg sim_standalone)" real_hardware="$(arg real_hardware)" finger_type="soft">
+    <xacro:wsg_50_xacro parent="base_link" finger_length="0.023" finger_tip="0.0" >
         <origin xyz="0 0 0.1" rpy="0 0 0"/>
     </xacro:wsg_50_xacro>

File: wsg_50_simulation/urdf/wsg_50.srdf.xacro (robot description, xacro)
@@ -7,16 +7,16 @@
     <xacro:macro name="weiss-wsg50_group_define" params="group_name prefix">
         <group name="${group_name}">
-            <link name="${prefix}_base"/>
-            <link name="${prefix}_mounting_plate"/>
-            <link name="${prefix}_base_link"/>
-            <link name="${prefix}_gripper_right"/>
-            <link name="${prefix}_gripper_left"/>
-            <link name="${prefix}_finger_left"/>
-            <link name="${prefix}_finger_right"/>
-            <link name="${prefix}_width"/>
-            <link name="${prefix}_center"/>
-            <joint name="${prefix}_joint"/>
-            <passive_joint name="${prefix}_base_joint_gripper_left"/>
-            <passive_joint name="${prefix}_base_joint_gripper_right"/>
+            <link name="base"/>
+            <link name="mounting_plate"/>
+            <link name="base_link"/>
+            <link name="gripper_right"/>
+            <link name="gripper_left"/>
+            <link name="finger_left"/>
+            <link name="finger_right"/>
+            <link name="width"/>
+            <link name="center"/>
+            <joint name="joint"/>
+            <passive_joint name="base_joint_gripper_left"/>
+            <passive_joint name="base_joint_gripper_right"/>
         </group>
         <group_state name="open" group="${group_name}">
@@ -32,27 +32,27 @@
     </xacro:macro>
     <xacro:macro name="weiss-wsg50_autocol" params="prefix">
-        <disable_collisions link1="${prefix}_mounting_plate" link2="${prefix}_base_link" reason="Adjacent"/>
-        <disable_collisions link1="${prefix}_mounting_plate" link2="${prefix}_gripper_right" reason="Never"/>
-        <disable_collisions link1="${prefix}_mounting_plate" link2="${prefix}_gripper_left" reason="Never"/>
-        <disable_collisions link1="${prefix}_mounting_plate" link2="${prefix}_finger_left" reason="Never"/>
-        <disable_collisions link1="${prefix}_mounting_plate" link2="${prefix}_finger_right" reason="Never"/>
-        <disable_collisions link1="${prefix}_base_link" link2="${prefix}_gripper_right" reason="Adjacent"/>
-        <disable_collisions link1="${prefix}_base_link" link2="${prefix}_gripper_left" reason="Adjacent"/>
-        <disable_collisions link1="${prefix}_base_link" link2="${prefix}_finger_left" reason="Never"/>
-        <disable_collisions link1="${prefix}_base_link" link2="${prefix}_finger_right" reason="Never"/>
-        <disable_collisions link1="${prefix}_gripper_right" link2="${prefix}_gripper_left" reason="Adjacent"/>
-        <disable_collisions link1="${prefix}_gripper_right" link2="${prefix}_finger_left" reason="Never"/>
-        <disable_collisions link1="${prefix}_gripper_right" link2="${prefix}_finger_right" reason="Adjacent"/>
-        <disable_collisions link1="${prefix}_gripper_left" link2="${prefix}_finger_left" reason="Adjacent"/>
-        <disable_collisions link1="${prefix}_gripper_left" link2="${prefix}_finger_right" reason="Never"/>
-        <disable_collisions link1="${prefix}_finger_left" link2="${prefix}_finger_right" reason="Adjacent"/>
+        <disable_collisions link1="mounting_plate" link2="base_link" reason="Adjacent"/>
+        <disable_collisions link1="mounting_plate" link2="gripper_right" reason="Never"/>
+        <disable_collisions link1="mounting_plate" link2="gripper_left" reason="Never"/>
+        <disable_collisions link1="mounting_plate" link2="finger_left" reason="Never"/>
+        <disable_collisions link1="mounting_plate" link2="finger_right" reason="Never"/>
+        <disable_collisions link1="base_link" link2="gripper_right" reason="Adjacent"/>
+        <disable_collisions link1="base_link" link2="gripper_left" reason="Adjacent"/>
+        <disable_collisions link1="base_link" link2="finger_left" reason="Never"/>
+        <disable_collisions link1="base_link" link2="finger_right" reason="Never"/>
+        <disable_collisions link1="gripper_right" link2="gripper_left" reason="Adjacent"/>
+        <disable_collisions link1="gripper_right" link2="finger_left" reason="Never"/>
+        <disable_collisions link1="gripper_right" link2="finger_right" reason="Adjacent"/>
+        <disable_collisions link1="gripper_left" link2="finger_left" reason="Adjacent"/>
+        <disable_collisions link1="gripper_left" link2="finger_right" reason="Never"/>
+        <disable_collisions link1="finger_left" link2="finger_right" reason="Adjacent"/>
     </xacro:macro>
     <xacro:macro name="weiss-wsg50_col_with" params="prefix link">
-        <disable_collisions link1="${prefix}_mounting_plate" link2="${link}" reason="Never"/>
-        <disable_collisions link1="${prefix}_base_link" link2="${link}" reason="Never"/>
-        <disable_collisions link1="${prefix}_gripper_right" link2="${link}" reason="Never"/>
-        <disable_collisions link1="${prefix}_gripper_left" link2="${link}" reason="Never"/>
-        <disable_collisions link1="${prefix}_finger_left" link2="${link}" reason="Never"/>
-        <disable_collisions link1="${prefix}_finger_right" link2="${link}" reason="Never"/>
+        <disable_collisions link1="mounting_plate" link2="${link}" reason="Never"/>
+        <disable_collisions link1="base_link" link2="${link}" reason="Never"/>
+        <disable_collisions link1="gripper_right" link2="${link}" reason="Never"/>
+        <disable_collisions link1="gripper_left" link2="${link}" reason="Never"/>
+        <disable_collisions link1="finger_left" link2="${link}" reason="Never"/>
+        <disable_collisions link1="finger_right" link2="${link}" reason="Never"/>
     </xacro:macro>
 </robot>

File: wsg_50_simulation/urdf/wsg_50.urdf (robot description, URDF)
Before this commit: robot wsg_50, 6 links, 5 joints
Joints:
- joint base_joint_gripper_right: mimic (none) -> joint=base_joint_gripper_left multiplier=-1 offset=0

File: wsg_50_simulation/urdf/wsg_50.urdf.xacro (robot description, xacro)
@@ -8,12 +8,12 @@
 <!-- finger_tip:    Offset of finger tip along fingers' motion direction.
                     Use e.g. for single contact point tip on finger. (default 0) -->
-<xacro:macro name="wsg_50_xacro" params="name parent finger_length finger_tip *origin">
- <joint name="${name}_anterior_gripper_joint" type="fixed">
+<xacro:macro name="wsg_50_xacro" params="parent finger_length finger_tip *origin">
+ <joint name="wsg_50_anterior_gripper_joint" type="fixed">
     <insert_block name="origin"/>
     <parent link="${parent}"/>
-    <child link="${name}_base_link"/>
+    <child link="wsg_50_base_link"/>
  </joint>
 <!-- BASE LINK -->
- <link name="${name}_base_link">
+ <link name="wsg_50_base_link">
       <inertial>
           <mass value="1.3" />
@@ -42,117 +42,117 @@
      </collision>
   </link>
-  <gazebo reference="${name}_base_link">
+  <gazebo reference="wsg_50_base_link">
     <material>Gazebo/Grey</material>
     <turnGravityOff>false</turnGravityOff>
   </gazebo>
-  <joint name="${name}_center_joint" type="fixed">
+  <joint name="wsg_50_center_joint" type="fixed">
      <origin xyz="0 0 ${finger_length}" rpy="0 0 0" />      <!--origin xyz="-0.0067 0 0.049" rpy="0 0 0" /-->
-     <parent link="${name}_base_link"/>
-     <child link="${name}_center" />
-  </joint>
-  <link name="${name}_center">
+     <parent link="wsg_50_base_link"/>
+     <child link="wsg_50_center" />
+  </joint>
+  <link name="wsg_50_center">
   </link>
   <!-- GRIPPER LEFT -->
-  <joint name="${name}_finger_left_joint" type="prismatic">
+  <joint name="wsg_50_finger_left_joint" type="prismatic">
      <limit lower="-0.055" upper="-0.0027" effort="1.0" velocity="1.0"/>
      <origin xyz="0 0 0" rpy="0 0 0" />      <!--origin xyz="-0.0067 0 0.049" rpy="0 0 0" /-->
-     <parent link="${name}_base_link"/>
-     <child link="${name}_gripper_left" />
+     <parent link="wsg_50_base_link"/>
+     <child link="wsg_50_gripper_left" />
      <dynamics friction="100" damping="100" />
      <axis xyz="1 0 0"/>
      <limit effort="100" velocity="100"/>
   </joint>
-  <transmission name="${name}_base_trans_left" type="pr2_mechanism_model/SimpleTransmission">
-     <actuator name="${name}_base_motor_left" />
-     <joint name="${name}_base_joint_gripper_left" />
+  <transmission name="wsg_50_base_trans_left" type="pr2_mechanism_model/SimpleTransmission">
+     <actuator name="wsg_50_base_motor_left" />
+     <joint name="wsg_50_base_joint_gripper_left" />
      <mechanicalReduction>1</mechanicalReduction>
      <motorTorqueConstant>1</motorTorqueConstant>
   </transmission>
-  <link name="${name}_gripper_left">
-      <inertial>
-          <mass value="0.1" />
-          <origin xyz="0 0 0" />
-      <inertia ixx="1.0" ixy="0.0" ixz="0.0"
-               iyy="1.0" iyz="0.0"
-               izz="1.0" />
-      </inertial>
-      <visual>
-          <origin xyz="0.0 0 0" rpy="0 0 0" />
-          <geometry>
-             <mesh filename="package://wsg_50_simulation/meshes/GUIDE_WSG50_110.stl" scale="0.001 0.001 0.001"/>
-	     <!--box size="0.0175 0.03 0.024"/-->
-          </geometry>
-          <material name="black">
-		<color rgba="0 0 0 0"/>
-      	  </material>
-      </visual>
-      <collision>
-          <origin xyz="0 0 0" rpy="0 0 0" />
-          <geometry>
-	     <!--box size="0.0175 0.03 0.024"/-->
-             <mesh filename="package://wsg_50_simulation/meshes/GUIDE_WSG50_110.stl" scale="0.001 0.001 0.001"/>
-         </geometry>
-     </collision>
-     <contact_coefficients kd="1.0" kp="1000.0" mu="0"/>
-  </link>
-  <gazebo reference="${name}_gripper_left">
+  <link name="wsg_50_gripper_left">
+      <inertial>
+          <mass value="0.1" />
+          <origin xyz="0 0 0" />
+      <inertia ixx="1.0" ixy="0.0" ixz="0.0"
+               iyy="1.0" iyz="0.0"
+               izz="1.0" />
+      </inertial>
+      <visual>
+          <origin xyz="0.0 0 0" rpy="0 0 0" />
+          <geometry>
+             <mesh filename="package://wsg_50_simulation/meshes/GUIDE_WSG50_110.stl" scale="0.001 0.001 0.001"/>
+	     <!--box size="0.0175 0.03 0.024"/-->
+          </geometry>
+          <material name="black">
+		<color rgba="0 0 0 0"/>
+      	  </material>
+      </visual>
+      <collision>
+          <origin xyz="0 0 0" rpy="0 0 0" />
+          <geometry>
+	     <!--box size="0.0175 0.03 0.024"/-->
+             <mesh filename="package://wsg_50_simulation/meshes/GUIDE_WSG50_110.stl" scale="0.001 0.001 0.001"/>
+         </geometry>
+     </collision>
+     <contact_coefficients kd="1.0" kp="1000.0" mu="0"/>
+  </link>
+  <gazebo reference="wsg_50_gripper_left">
     <material>Gazebo/Blue</material>
     <turnGravityOff>false</turnGravityOff>
   </gazebo>
   <!-- LEFT FINGER -->
-  <joint name="${name}_guide_joint_finger_left" type="fixed">
+  <joint name="wsg_50_guide_joint_finger_left" type="fixed">
      <origin xyz="${finger_tip} 0 ${finger_length}" rpy="0 0 0" />
-     <parent link="${name}_gripper_left"/>
-     <child link="${name}_finger_left" />
+     <parent link="wsg_50_gripper_left"/>
+     <child link="wsg_50_finger_left" />
      <dynamics friction="100" damping="100" />
      <axis xyz="1 0 0"/>
      <limit effort="100" velocity="100"/>
   </joint>
-  <link name="${name}_finger_left">
-      <inertial>
-          <mass value="0.1" />
-          <origin xyz="0 0 0" />
-      <inertia ixx="1.0" ixy="0.0" ixz="0.0"
-               iyy="1.0" iyz="0.0"
-               izz="1.0" />
-      </inertial>
-      <visual>
-          <origin xyz="0.0 0 0" rpy="0 0 0" />
-          <geometry>
-             <mesh filename="package://wsg_50_simulation/meshes/WSG-FMF.stl" scale="0.001 0.001 0.001"/>
-          </geometry>
-          <material name="black">
-		<color rgba="0 0 0 0"/>
-      	  </material>
-      </visual>
-      <collision>
-          <origin xyz="0 0 0" rpy="0 0 0" />
-          <geometry>
-             <mesh filename="package://wsg_50_simulation/meshes/WSG-FMF.stl" scale="0.001 0.001 0.001"/>
-         </geometry>
-     </collision>
-     <contact_coefficients kd="1.0" kp="1000.0" mu="0"/>
-  </link>
-  <gazebo reference="${name}_finger_left">
+  <link name="wsg_50_finger_left">
+      <inertial>
+          <mass value="0.1" />
+          <origin xyz="0 0 0" />
+      <inertia ixx="1.0" ixy="0.0" ixz="0.0"
+               iyy="1.0" iyz="0.0"
+               izz="1.0" />
+      </inertial>
+      <visual>
+          <origin xyz="0.0 0 0" rpy="0 0 0" />
+          <geometry>
+             <mesh filename="package://wsg_50_simulation/meshes/WSG-FMF.stl" scale="0.001 0.001 0.001"/>
+          </geometry>
+          <material name="black">
+		<color rgba="0 0 0 0"/>
+      	  </material>
+      </visual>
+      <collision>
+          <origin xyz="0 0 0" rpy="0 0 0" />
+          <geometry>
+             <mesh filename="package://wsg_50_simulation/meshes/WSG-FMF.stl" scale="0.001 0.001 0.001"/>
+         </geometry>
+     </collision>
+     <contact_coefficients kd="1.0" kp="1000.0" mu="0"/>
+  </link>
+  <gazebo reference="wsg_50_finger_left">
     <material>Gazebo/Blue</material>
     <turnGravityOff>false</turnGravityOff>
   </gazebo>
   <!-- GRIPPER RIGHT -->
-  <joint name="${name}_finger_right_joint" type="prismatic">
+  <joint name="wsg_50_finger_right_joint" type="prismatic">
      <limit lower="0.0027" upper="0.055" effort="1.0" velocity="1.0"/>
      <origin xyz="0 0 0" rpy="0 0 3.14159" />
-     <parent link="${name}_base_link"/>
-     <child link="${name}_gripper_right" />
+     <parent link="wsg_50_base_link"/>
+     <child link="wsg_50_gripper_right" />
      <axis xyz="-1 0 0"/>
      <dynamics friction="100" damping="100" />
      <limit effort="100" velocity="100"/>
   </joint>
-  <transmission name="${name}_base_trans_right" type="pr2_mechanism_model/SimpleTransmission">
-     <actuator name="${name}_base_motor_right" />
-     <joint name="${name}_base_joint_gripper_right" />
+  <transmission name="wsg_50_base_trans_right" type="pr2_mechanism_model/SimpleTransmission">
+     <actuator name="wsg_50_base_motor_right" />
+     <joint name="wsg_50_base_joint_gripper_right" />
      <mechanicalReduction>1</mechanicalReduction>
      <motorTorqueConstant>1</motorTorqueConstant>
   </transmission>
-    <link name="${name}_gripper_right">
+    <link name="wsg_50_gripper_right">
       <inertial>
           <mass value="0.1" />
@@ -186,38 +186,38 @@
   </gazebo>
   <!-- RIGHT FINGER -->
-  <joint name="${name}_guide_joint_finger_right" type="fixed">
+  <joint name="wsg_50_guide_joint_finger_right" type="fixed">
      <origin xyz="${finger_tip} 0 ${finger_length}" rpy="0 0 0" />
-     <parent link="${name}_gripper_right"/>
-     <child link="${name}_finger_right" />
+     <parent link="wsg_50_gripper_right"/>
+     <child link="wsg_50_finger_right" />
      <dynamics friction="100" damping="100" />
      <axis xyz="1 0 0"/>
      <limit effort="100" velocity="100"/>
   </joint>
-  <link name="${name}_finger_right">
-      <inertial>
-          <mass value="0.1" />
-          <origin xyz="0 0 0" />
-      <inertia ixx="1.0" ixy="0.0" ixz="0.0"
-               iyy="1.0" iyz="0.0"
-               izz="1.0" />
-      </inertial>
-      <visual>
-          <origin xyz="0.0 0 0" rpy="0 0 0" />
-          <geometry>
-             <mesh filename="package://wsg_50_simulation/meshes/WSG-FMF.stl" scale="0.001 0.001 0.001"/>
-          </geometry>
-          <material name="black">
-		<color rgba="0 0 0 0"/>
-      	  </material>
-      </visual>
-      <collision>
-          <origin xyz="0 0 0" rpy="0 0 0" />
-          <geometry>
-             <mesh filename="package://wsg_50_simulation/meshes/WSG-FMF.stl" scale="0.001 0.001 0.001"/>
-         </geometry>
-     </collision>
-     <contact_coefficients kd="1.0" kp="1000.0" mu="0"/>
-  </link>
-  <gazebo reference="${name}_finger_right">
+  <link name="wsg_50_finger_right">
+      <inertial>
+          <mass value="0.1" />
+          <origin xyz="0 0 0" />
+      <inertia ixx="1.0" ixy="0.0" ixz="0.0"
+               iyy="1.0" iyz="0.0"
+               izz="1.0" />
+      </inertial>
+      <visual>
+          <origin xyz="0.0 0 0" rpy="0 0 0" />
+          <geometry>
+             <mesh filename="package://wsg_50_simulation/meshes/WSG-FMF.stl" scale="0.001 0.001 0.001"/>
+          </geometry>
+          <material name="black">
+		<color rgba="0 0 0 0"/>
+      	  </material>
+      </visual>
+      <collision>
+          <origin xyz="0 0 0" rpy="0 0 0" />
+          <geometry>
+             <mesh filename="package://wsg_50_simulation/meshes/WSG-FMF.stl" scale="0.001 0.001 0.001"/>
+         </geometry>
+     </collision>
+     <contact_coefficients kd="1.0" kp="1000.0" mu="0"/>
+  </link>
+  <gazebo reference="wsg_50_finger_right">
     <material>Gazebo/White</material>
     <turnGravityOff>false</turnGravityOff>
